File: EsquematicoPractica1.sch (EAGLE design)
At the start: 57 parts, among them IC1 GSOT05C-GS08, J1 M50-3500542, Q1 IRF7416PBF, Q2 IRF7416PBF, U1 MKL27Z64VLH4, U2 SFH6156-4TSMD-4_VO-L, U3 MC34063ADR, U4 SFH6156-4TSMD-4_VO-L, U5 SFH6156-4TSMD-4_VO-L, U6 SFH6156-4TSMD-4_VO-L, U7 TLV274QPWRG4Q1, X1 MINI-USB-SCHIELD-32005-201, Y3 32.768KHZ

Commit message: RST & LED Polarización PERFECTO
Verificar las resistencias usadas para las entradas y salidad además de empezar a hacer conexiones directamente con la KL27z
Parts:
- removed R14: 220, rcl:R-US_M1206
- added C5, C6: C0402C104K8PAC, C0402C104K8PAC:C0402C104K8PAC
- added R15: RK73B1JTTD221J, RK73B1JTTD221J:RK73B1JTTD221J
- S1: value RDT1034 -> EVQPE105K; device switch:RDT1034 -> EVQPE105K:EVQPE105K
Connections:
- new net +3V3: C5.2
- new net PTA20: C5.1, C6.2, S1.2, U1.PTA20
- net +5V: no longer R14.2
- net GND: now also C6.1, S1.1
- net N$26: now also R15.1; no longer R14.1
Other:
- moved on the sheet: LED3
Changed lines of the file:
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@@
 <?xml version="1.0" encoding="utf-8"?>
 <!DOCTYPE eagle SYSTEM "eagle.dtd">
-<eagle version="8.6.0">
+<eagle version="8.6.2">
 <drawing>
 <settings>
@@
 <part name="R81" library="RK73H1JLTD1005F" deviceset="RK73H1JLTD1005F" device="" value="10M"/>
 <part name="U7" library="TLV274QPWRG4Q1" deviceset="TLV274QPWRG4Q1" device=""/>
-<part name="SUPPLY2" library="supply2" library_urn="urn:adsk.eagle:library:372" deviceset="+5V" device="" value="+3V3"/>
-<part name="R14" library="rcl" library_urn="urn:adsk.eagle:library:334" deviceset="R-US_" device="M1206" package3d_urn="urn:adsk.eagle:package:23566/1" value="220"/>
 <part name="LED3" library="led" library_urn="urn:adsk.eagle:library:259" deviceset="LED" device="5MM" package3d_urn="urn:adsk.eagle:package:15799/2"/>
 <part name="GND12" library="supply1" library_urn="urn:adsk.eagle:library:371" deviceset="GND" device=""/>
-<part name="S1" library="switch" library_urn="urn:adsk.eagle:library:380" deviceset="RDT1034" device="" package3d_urn="urn:adsk.eagle:package:27704/1"/>
+<part name="S1" library="EVQPE105K" deviceset="EVQPE105K" device=""/>
+<part name="GND13" library="supply1" library_urn="urn:adsk.eagle:library:371" deviceset="GND" device=""/>
+<part name="GND14" library="supply1" library_urn="urn:adsk.eagle:library:371" deviceset="GND" device=""/>
+<part name="C5" library="C0402C104K8PAC" deviceset="C0402C104K8PAC" device=""/>
+<part name="C6" library="C0402C104K8PAC" deviceset="C0402C104K8PAC" device=""/>
+<part name="R15" library="RK73B1JTTD221J" deviceset="RK73B1JTTD221J" device=""/>
 </parts>
 <sheets>
@@
 <wire x1="-5.08" y1="-78.74" x2="-15.24" y2="-78.74" width="0.1524" layer="97"/>
 <wire x1="-15.24" y1="-78.74" x2="-15.24" y2="-15.24" width="0.1524" layer="97"/>
-<wire x1="33.02" y1="-101.6" x2="-12.5476" y2="-101.6" width="0.1524" layer="97"/>
-<wire x1="33.02" y1="-165.1" x2="33.02" y2="-101.6" width="0.1524" layer="97"/>
-<wire x1="33.02" y1="-165.1" x2="-2.3876" y2="-165.1" width="0.1524" layer="97"/>
-<wire x1="-2.54" y1="-165.1" x2="-12.7" y2="-165.1" width="0.1524" layer="97"/>
-<wire x1="-12.7" y1="-165.1" x2="-12.7" y2="-101.6" width="0.1524" layer="97"/>
+<wire x1="33.02" y1="-104.14" x2="-12.5476" y2="-104.14" width="0.1524" layer="97"/>
+<wire x1="33.02" y1="-170.18" x2="33.02" y2="-104.14" width="0.1524" layer="97"/>
+<wire x1="33.02" y1="-170.18" x2="-2.3876" y2="-170.18" width="0.1524" layer="97"/>
+<wire x1="-2.54" y1="-170.18" x2="-12.7" y2="-170.18" width="0.1524" layer="97"/>
+<wire x1="-12.7" y1="-170.18" x2="-12.7" y2="-104.14" width="0.1524" layer="97"/>
 <text x="-10.16" y="-99.06" size="1.778" layer="97">LED indicador de polarización</text>
-<wire x1="124.46" y1="-99.06" x2="78.8924" y2="-99.06" width="0.1524" layer="97"/>
-<wire x1="124.46" y1="-162.56" x2="124.46" y2="-99.06" width="0.1524" layer="97"/>
-<wire x1="124.46" y1="-162.56" x2="89.0524" y2="-162.56" width="0.1524" layer="97"/>
-<wire x1="88.9" y1="-162.56" x2="78.74" y2="-162.56" width="0.1524" layer="97"/>
-<wire x1="78.74" y1="-162.56" x2="78.74" y2="-99.06" width="0.1524" layer="97"/>
-<text x="81.28" y="-96.52" size="1.778" layer="97">Pulsador de RST</text>
+<wire x1="170.18" y1="-91.44" x2="78.8924" y2="-91.44" width="0.1524" layer="97"/>
+<wire x1="170.18" y1="-170.18" x2="170.18" y2="-91.44" width="0.1524" layer="97"/>
+<wire x1="170.18" y1="-170.18" x2="78.8924" y2="-170.18" width="0.1524" layer="97"/>
+<wire x1="78.74" y1="-170.18" x2="78.74" y2="-91.44" width="0.1524" layer="97"/>
+<text x="81.28" y="-86.36" size="1.778" layer="97">Pulsador de RST</text>
 </plain>
 <instances>
@@
 <instance part="OUT2" gate="-1" x="129.54" y="-55.88" rot="R180"/>
 <instance part="3.3V1" gate="-1" x="114.3" y="-27.94" rot="R270"/>
-<instance part="SUPPLY2" gate="+5V" x="5.08" y="-116.84" smashed="yes">
-<attribute name="VALUE" x="3.175" y="-118.745" size="1.778" layer="96" rot="R90"/>
-</instance>
-<instance part="R14" gate="G$1" x="5.08" y="-132.08" rot="R90"/>
-<instance part="LED3" gate="G$1" x="5.08" y="-144.78"/>
-<instance part="GND12" gate="1" x="5.08" y="-157.48"/>
-<instance part="S1" gate="G$1" x="96.52" y="-121.92"/>
+<instance part="LED3" gate="G$1" x="5.08" y="-152.4"/>
+<instance part="GND12" gate="1" x="5.08" y="-162.56"/>
+<instance part="S1" gate="G$1" x="99.06" y="-129.54"/>
+<instance part="GND13" gate="1" x="91.44" y="-147.32"/>
+<instance part="GND14" gate="1" x="137.16" y="-160.02"/>
+<instance part="C5" gate="G$1" x="137.16" y="-124.46" rot="R90"/>
+<instance part="C6" gate="G$1" x="137.16" y="-152.4" rot="R90"/>
+<instance part="R15" gate="G$1" x="5.08" y="-144.78" rot="R90"/>
 </instances>
 <busses>
@@
 <pinref part="GND12" gate="1" pin="GND"/>
 <pinref part="LED3" gate="G$1" pin="C"/>
-<wire x1="5.08" y1="-154.94" x2="5.08" y2="-149.86" width="0.1524" layer="91"/>
+<wire x1="5.08" y1="-160.02" x2="5.08" y2="-157.48" width="0.1524" layer="91"/>
+</segment>
+<segment>
+<pinref part="GND13" gate="1" pin="GND"/>
+<wire x1="91.44" y1="-144.78" x2="91.44" y2="-129.54" width="0.1524" layer="91"/>
+<pinref part="S1" gate="G$1" pin="1"/>
+<wire x1="91.44" y1="-129.54" x2="99.06" y2="-129.54" width="0.1524" layer="91"/>
+</segment>
+<segment>
+<pinref part="C6" gate="G$1" pin="1"/>
+<pinref part="GND14" gate="1" pin="GND"/>
+<wire x1="137.16" y1="-152.4" x2="137.16" y2="-157.48" width="0.1524" layer="91"/>
 </segment>
 </net>
@@
 <pinref part="SUPPLY1" gate="+5V" pin="+5V"/>
 </segment>
-<segment>
-<pinref part="R14" gate="G$1" pin="2"/>
-<pinref part="SUPPLY2" gate="+5V" pin="+5V"/>
-<wire x1="5.08" y1="-127" x2="5.08" y2="-119.38" width="0.1524" layer="91"/>
-</segment>
 </net>
 <net name="N$1" class="0">
@@
 <segment>
 <pinref part="LED3" gate="G$1" pin="A"/>
-<pinref part="R14" gate="G$1" pin="1"/>
-<wire x1="5.08" y1="-142.24" x2="5.08" y2="-137.16" width="0.1524" layer="91"/>
-</segment>
-</net>
+<wire x1="5.08" y1="-149.86" x2="5.08" y2="-144.78" width="0.1524" layer="91"/>
+<pinref part="R15" gate="G$1" pin="1"/>
+</segment>
+</net>
+<net name="PTA20" class="0">
+<segment>
+<pinref part="U1" gate="A" pin="PTA20"/>
+<wire x1="144.78" y1="226.06" x2="157.48" y2="226.06" width="0.1524" layer="91"/>
+<wire x1="160.02" y1="226.06" x2="157.48" y2="226.06" width="0.1524" layer="91"/>
+<label x="165.1" y="226.06" size="1.778" layer="95"/>
+</segment>
+<segment>
+<pinref part="S1" gate="G$1" pin="2"/>
+<wire x1="119.38" y1="-129.54" x2="137.16" y2="-129.54" width="0.1524" layer="91"/>
+<pinref part="C6" gate="G$1" pin="2"/>
+<wire x1="137.16" y1="-129.54" x2="137.16" y2="-139.7" width="0.1524" layer="91"/>
+<pinref part="C5" gate="G$1" pin="1"/>
+<wire x1="137.16" y1="-129.54" x2="137.16" y2="-124.46" width="0.1524" layer="91"/>
+<junction x="137.16" y="-129.54"/>
+<wire x1="137.16" y1="-129.54" x2="144.78" y2="-129.54" width="0.1524" layer="91"/>
+<label x="147.32" y="-129.54" size="1.778" layer="95"/>
+</segment>
+</net>
+<net name="+3V3" class="0">
+<segment>
+<pinref part="C5" gate="G$1" pin="2"/>
+<wire x1="137.16" y1="-111.76" x2="137.16" y2="-104.14" width="0.1524" layer="91"/>
+<label x="137.16" y="-101.6" size="1.778" layer="95"/>
+</segment>
+<segment>
+<wire x1="5.08" y1="-127" x2="5.08" y2="-119.38" width="0.1524" layer="91"/>
+<label x="5.08" y="-116.84" size="1.778" layer="95"/>
+</segment>
+</net>

Commit message: Merge bot schematics
Parts:
- removed L3, L4: MPZ2012S331A, MPZ2012S331AT000:MPZ2012S331AT000
- removed U7: TLV274QPWRG4Q1, TLV274QPWRG4Q1:TLV274QPWRG4Q1
- added L5, L6: MPZ2012S331A, MPZ2012S331AT000:MPZ2012S331AT000
- added R103: 6.7K, rcl:R-US_M1206
- added R104: 3.3K, rcl:R-US_M1206
- added R105, R106: 33, rcl:R-US_M1206
- added U13: TLV274QPWRG4Q1, TLV274QPWRG4Q1:TLV274QPWRG4Q1
- R100, R101: device rcl:R-US_M1206 -> RC0402FR-0733RL:RC0402FR-0733RL
Connections:
- net N$34 renamed SDA_JTAG_TMS
- net N$35 renamed EXTAL_32KHZ
- net N$36 renamed SDA_JTAG_TCLK
- net N$37 renamed SDA_JTAG_TDO
- net N$38 renamed SDA_JTAG_TDI
- net N$39 renamed SDA_RST_B
- removed net N$27: IC1.CATHODE(2), R100.1, X1G$1.3
- removed net N$29: IC1.CATHODE(1), R101.2, X1G$1.2
- removed net N$30: L3.1, X1G$1.1
- removed net N$31: L4.1, X1S.S1, X1S.S2, X1S.S3, X1S.S4
- removed net N$32: R100.2
- removed net N$33: R101.1
- removed net N$40: J1.1
- removed net N$41: C43.1, Y3.4
- new net N$71: IC1.CATHODE(2), R101.1, X1G$1.3
- new net N$72: L5.1, X1G$1.1
- new net N$73: IC1.CATHODE(1), R100.1, X1G$1.2
- new net N$74: L6.1, X1S.S1, X1S.S2, X1S.S3, X1S.S4
- new net N$75: U13.2IN-, U13.2OUT
- new net N$76: R103.2, R104.2, U13.2IN+
- new net N$77: U13.4IN-, U13.4OUT
- new net N$78: R105.2, R106.2, U13.4IN+
- new net P3V3_SDA: J1.1, R102.2
- new net P5V_SDA: L5.2, TP5.1
- new net USB_DM: R100.2, U1.USB0_DM
- new net USB_DP: R101.2, U1.USB0_DP
- new net XTAL_32KHZ: C43.1, R81.2, Y3.4
- net GND: now also L6.2, R104.1, R106.1; no longer L4.2
- net N$26: no longer L3.2, TP5.1
Other:
- note added: "2 ENTRADAS 0-10 V CON AISLAMIENTO DE IMPEDANCIAS"
- note added: "32KHz CLK"
- note added: "MINI-USB-B"
- note added: "OpenSDA INTERFACE JTAG CONNECTOR"

Commit message: Update resistors
Parts:
- R10: value (none) -> 300
- R11, R8, R9: value (none) -> 300; device rcl:R-US_0204/7 -> rcl:R-US_0309/12
Changed lines of the file:
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@@
 <part name="U6" library="SFH6156-4T" deviceset="SFH6156-4T" device="SMD-4_VO-L"/>
 <part name="INPUT1" library="con-ptr500" library_urn="urn:adsk.eagle:library:181" deviceset="AK300/2" device="" package3d_urn="urn:adsk.eagle:package:9881/1"/>
-<part name="R10" library="rcl" library_urn="urn:adsk.eagle:library:334" deviceset="R-US_" device="0204/7" package3d_urn="urn:adsk.eagle:package:23498/1"/>
-<part name="R11" library="rcl" library_urn="urn:adsk.eagle:library:334" deviceset="R-US_" device="0204/7" package3d_urn="urn:adsk.eagle:package:23498/1"/>
+<part name="R10" library="rcl" library_urn="urn:adsk.eagle:library:334" deviceset="R-US_" device="0204/7" package3d_urn="urn:adsk.eagle:package:23498/1" value="300"/>
+<part name="R11" library="rcl" library_urn="urn:adsk.eagle:library:334" deviceset="R-US_" device="0309/12" package3d_urn="urn:adsk.eagle:package:23571/1" value="300"/>
 <part name="LED1" library="led" library_urn="urn:adsk.eagle:library:259" deviceset="LED" device="5MM" package3d_urn="urn:adsk.eagle:package:15799/2"/>
 <part name="GND8" library="supply1" library_urn="urn:adsk.eagle:library:371" deviceset="GND" device=""/>
@@
 <part name="U5" library="SFH6156-4T" deviceset="SFH6156-4T" device="SMD-4_VO-L"/>
 <part name="INPUT2" library="con-ptr500" library_urn="urn:adsk.eagle:library:181" deviceset="AK300/2" device="" package3d_urn="urn:adsk.eagle:package:9881/1"/>
-<part name="R8" library="rcl" library_urn="urn:adsk.eagle:library:334" deviceset="R-US_" device="0204/7" package3d_urn="urn:adsk.eagle:package:23498/1"/>
-<part name="R9" library="rcl" library_urn="urn:adsk.eagle:library:334" deviceset="R-US_" device="0204/7" package3d_urn="urn:adsk.eagle:package:23498/1"/>
+<part name="R8" library="rcl" library_urn="urn:adsk.eagle:library:334" deviceset="R-US_" device="0309/12" package3d_urn="urn:adsk.eagle:package:23571/1" value="300"/>
+<part name="R9" library="rcl" library_urn="urn:adsk.eagle:library:334" deviceset="R-US_" device="0309/12" package3d_urn="urn:adsk.eagle:package:23571/1" value="300"/>
 <part name="LED2" library="led" library_urn="urn:adsk.eagle:library:259" deviceset="LED" device="5MM" package3d_urn="urn:adsk.eagle:package:15799/2"/>
 <part name="GND10" library="supply1" library_urn="urn:adsk.eagle:library:371" deviceset="GND" device=""/>
