File: EsquematicoPractica1.sch (EAGLE design)
At the start: 129 parts, among them IC1 GSOT05C-GS08, IC10 NCP1117ST33T3G, IC2 RCV420JP, IC3 TC7662BEOA, IC4 MC7812BTG, IC5 RCV420JP, IC6 TC7662BEOA, IC7 MC7812BTG, IC8 GSOT05C-GS08, J2 M50-3500542, J3 M50-3500542, Q1 IRF7416PBF, Q2 IRF7416PBF, U1 MKL27Z64VLH4, U10 74LVC125AD, U13 TLV274QPWRG4Q1, U2 SFH6156-4TSMD-4_VO-L, U3 MC34063ADR, U4 SFH6156-4TSMD-4_VO-L, U5 SFH6156-4TSMD-4_VO-L, U6 SFH6156-4TSMD-4_VO-L, U7 MK20DX128VFM5, U8 74LVC125AD, U9 74LVC125AD, X1 MINI-USB-SCHIELD-32005-201, X2 MINI-USB-SCHIELD-32005-201, Y1 ABM3B-8.000MHZ-B2-T, Y3 32.768KHZ

Commit message: Esquemático Full Ahora Sí de Verdad
Valores y conexiones perfectas.
Connections:
- net +3V3: now also U1.VDD, U1.VDD_2, U1.VDD_3
- net +5V: no longer U1.VDD, U1.VDD_2, U1.VDD_3
Changed lines of the file:
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@@
 <?xml version="1.0" encoding="utf-8"?>
 <!DOCTYPE eagle SYSTEM "eagle.dtd">
-<eagle version="8.6.0">
+<eagle version="8.6.2">
 <drawing>
 <settings>
@@
 <part name="GND45" library="supply1" library_urn="urn:adsk.eagle:library:371" deviceset="GND" device=""/>
 <part name="JP4" library="pinhead" library_urn="urn:adsk.eagle:library:325" deviceset="PINHD-1X2" device="/90" package3d_urn="urn:adsk.eagle:package:22437/2"/>
-<part name="SUPPLY7" library="supply2" library_urn="urn:adsk.eagle:library:372" deviceset="+5V" device="" value="+3V3"/>
-<part name="SUPPLY8" library="supply2" library_urn="urn:adsk.eagle:library:372" deviceset="+5V" device="" value="+3V3"/>
-<part name="SUPPLY9" library="supply2" library_urn="urn:adsk.eagle:library:372" deviceset="+5V" device="" value="+3V3"/>
 <part name="IC9" library="v-reg" library_urn="urn:adsk.eagle:library:409" deviceset="78XXL" device="" package3d_urn="urn:adsk.eagle:package:30361/1"/>
 <part name="SUPPLY10" library="supply2" library_urn="urn:adsk.eagle:library:372" deviceset="VCC" device=""/>
@@
 <instance part="GND45" gate="1" x="665.48" y="-25.4"/>
 <instance part="JP4" gate="G$1" x="718.82" y="5.08" rot="R90"/>
-<instance part="SUPPLY7" gate="+5V" x="157.48" y="314.96" smashed="yes" rot="R90">
-<attribute name="VALUE" x="159.385" y="313.055" size="1.778" layer="96" rot="R180"/>
-</instance>
-<instance part="SUPPLY8" gate="+5V" x="167.64" y="246.38" smashed="yes" rot="R90">
-<attribute name="VALUE" x="169.545" y="244.475" size="1.778" layer="96" rot="R180"/>
-</instance>
-<instance part="SUPPLY9" gate="+5V" x="297.18" y="279.4" smashed="yes" rot="R270">
-<attribute name="VALUE" x="295.275" y="281.305" size="1.778" layer="96"/>
-</instance>
 <instance part="IC9" gate="A" x="-76.2" y="177.8"/>
 <instance part="SUPPLY10" gate="G$1" x="-101.6" y="177.8" smashed="yes" rot="R90">
@@
 </segment>
 <segment>
-<pinref part="U1" gate="A" pin="VDD_2"/>
-<pinref part="SUPPLY7" gate="+5V" pin="+5V"/>
-<wire x1="160.02" y1="314.96" x2="175.26" y2="314.96" width="0.1524" layer="91"/>
-</segment>
-<segment>
-<pinref part="U1" gate="A" pin="VDD_3"/>
-<pinref part="SUPPLY8" gate="+5V" pin="+5V"/>
-<wire x1="175.26" y1="246.38" x2="170.18" y2="246.38" width="0.1524" layer="91"/>
-</segment>
-<segment>
-<pinref part="U1" gate="A" pin="VDD"/>
-<pinref part="SUPPLY9" gate="+5V" pin="+5V"/>
-<wire x1="287.02" y1="279.4" x2="294.64" y2="279.4" width="0.1524" layer="91"/>
-</segment>
-<segment>
 <pinref part="IC9" gate="A" pin="OUT"/>
 <pinref part="+5V" gate="1" pin="+5V"/>
@@
 <label x="-71.12" y="-134.62" size="1.778" layer="95"/>
 </segment>
-</net>
+<segment>
+<pinref part="U1" gate="A" pin="VDD_2"/>
+<wire x1="160.02" y1="314.96" x2="175.26" y2="314.96" width="0.1524" layer="91"/>
+<label x="160.02" y="314.96" size="1.778" layer="95"/>
+</segment>
+<segment>
+<pinref part="U1" gate="A" pin="VDD_3"/>
+<wire x1="175.26" y1="246.38" x2="170.18" y2="246.38" width="0.1524" layer="91"/>
+<label x="167.64" y="246.38" size="1.778" layer="95"/>
+<label x="167.64" y="246.38" size="1.778" layer="95"/>
+</segment>
+<segment>
+<pinref part="U1" gate="A" pin="VDD"/>
+<wire x1="287.02" y1="279.4" x2="294.64" y2="279.4" width="0.1524" layer="91"/>
+<label x="294.64" y="279.4" size="1.778" layer="95"/>
+</segment>
+</net>

Commit message: Practica 1 - Total Entrega
PCB + Esquematico
Parts:
- removed U$1: MIKROE_CLICKMINI, mikrobus_lib:MIKROE_CLICKMINI
- added U11: MIKROE-971, MIKROE-971:MIKROE-971
Connections:
- net +3V3: now also U11.3V3; no longer U$1.3V3
- net +5V: now also U11.5V; no longer U$1.5V
- net GND: now also U11.GND(1), U11.GND(2); no longer U$1.GND1, U$1.GND2
- net I2C0_SCL: now also U11.SCL; no longer U$1.SCL
- net I2C0_SDA: now also U11.SDA; no longer U$1.SDA
- net LPUART0_RX_MKB: now also U11.RX; no longer U$1.RX
- net LPUART0_TX_MKB: now also U11.TX; no longer U$1.TX
- net PIN_INT: now also U11.INT; no longer U$1.INT
- net PTA20_RST: now also U11.RST; no longer U$1.RST
- net PTE20_A0: now also U11.AN; no longer U$1.AN
- net SPI0_MISO: now also U11.SDO; no longer U$1.MISO
- net SPI0_MOSI: now also U11.SDI; no longer U$1.MOSI
- net SPI0_PCS0: now also U11.CS; no longer U$1.CS
- net SPI0_SCK: now also U11.SCK; no longer U$1.SCK
- net TPM0_CH2_PWM: no longer U$1.PWM
Changed lines of the file:
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@@
 <part name="R101" library="RC0402FR-0733RL" deviceset="RC0402FR-0733RL" device="" value="33"/>
 <part name="R100" library="RC0402FR-0733RL" deviceset="RC0402FR-0733RL" device="" value="33"/>
-<part name="U$1" library="mikrobus_lib" deviceset="MIKROE_CLICK" device="MINI"/>
 <part name="IC2" library="RCV420JP" deviceset="RCV420JP" device=""/>
 <part name="IC3" library="TC7662BEOA" deviceset="TC7662BEOA" device=""/>
@@
 <part name="GND11" library="supply1" library_urn="urn:adsk.eagle:library:371" deviceset="GND" device=""/>
 <part name="GND49" library="supply1" library_urn="urn:adsk.eagle:library:371" deviceset="GND" device=""/>
+<part name="U11" library="MIKROE-971" deviceset="MIKROE-971" device=""/>
 </parts>
 <sheets>
@@
 <instance part="R101" gate="G$1" x="353.06" y="119.38"/>
 <instance part="R100" gate="G$1" x="358.14" y="109.22"/>
-<instance part="U$1" gate="G$1" x="-33.02" y="-119.38"/>
 <instance part="IC2" gate="G$1" x="-254" y="-198.12"/>
 <instance part="IC3" gate="G$1" x="-134.62" y="-238.76"/>
@@
 <instance part="GND11" gate="1" x="370.84" y="-327.66"/>
 <instance part="GND49" gate="1" x="429.26" y="-327.66"/>
+<instance part="U11" gate="G$1" x="-53.34" y="-104.14"/>
 </instances>
 <busses>
@@
 </segment>
 <segment>
-<pinref part="U$1" gate="G$1" pin="GND1"/>
-<wire x1="-53.34" y1="-139.7" x2="-68.58" y2="-139.7" width="0.1524" layer="91"/>
-<label x="-68.58" y="-139.7" size="1.778" layer="95"/>
-</segment>
-<segment>
-<pinref part="U$1" gate="G$1" pin="GND2"/>
-<wire x1="-15.24" y1="-139.7" x2="0" y2="-139.7" width="0.1524" layer="91"/>
-<label x="0" y="-139.7" size="1.778" layer="95"/>
+<wire x1="-53.34" y1="-121.92" x2="-73.66" y2="-121.92" width="0.1524" layer="91"/>
+<label x="-73.66" y="-121.92" size="1.778" layer="95"/>
+<pinref part="U11" gate="G$1" pin="GND(1)"/>
+</segment>
+<segment>
+<wire x1="-20.32" y1="-104.14" x2="0" y2="-104.14" width="0.1524" layer="91"/>
+<label x="0" y="-104.14" size="1.778" layer="95"/>
+<pinref part="U11" gate="G$1" pin="GND(2)"/>
 </segment>
 <segment>
@@
 </segment>
 <segment>
-<pinref part="U$1" gate="G$1" pin="5V"/>
-<wire x1="-15.24" y1="-134.62" x2="0" y2="-134.62" width="0.1524" layer="91"/>
-<label x="0" y="-134.62" size="1.778" layer="95"/>
+<wire x1="-20.32" y1="-106.68" x2="0" y2="-106.68" width="0.1524" layer="91"/>
+<label x="0" y="-106.68" size="1.778" layer="95"/>
+<pinref part="U11" gate="G$1" pin="5V"/>
 </segment>
 </net>
@@
 </segment>
 <segment>
-<pinref part="U$1" gate="G$1" pin="3V3"/>
-<wire x1="-53.34" y1="-134.62" x2="-68.58" y2="-134.62" width="0.1524" layer="91"/>
-<label x="-71.12" y="-134.62" size="1.778" layer="95"/>
+<wire x1="-53.34" y1="-119.38" x2="-73.66" y2="-119.38" width="0.1524" layer="91"/>
+<label x="-73.66" y="-119.38" size="1.778" layer="95"/>
+<pinref part="U11" gate="G$1" pin="3V3"/>
 </segment>
 <segment>
@@
 <net name="PTA20_RST" class="0">
 <segment>
-<pinref part="U$1" gate="G$1" pin="RST"/>
-<wire x1="-53.34" y1="-109.22" x2="-68.58" y2="-109.22" width="0.1524" layer="91"/>
-<label x="-73.66" y="-109.22" size="1.778" layer="95"/>
+<label x="-73.66" y="-106.68" size="1.778" layer="95"/>
+<wire x1="-73.66" y1="-106.68" x2="-53.34" y2="-106.68" width="0.1524" layer="91"/>
+<pinref part="U11" gate="G$1" pin="RST"/>
 </segment>
 </net>
@@
 </segment>
 <segment>
-<pinref part="U$1" gate="G$1" pin="AN"/>
 <wire x1="-53.34" y1="-104.14" x2="-73.66" y2="-104.14" width="0.1524" layer="91"/>
 <label x="-73.66" y="-104.14" size="1.778" layer="95"/>
+<pinref part="U11" gate="G$1" pin="AN"/>
 </segment>
 </net>
 <net name="SPI0_MISO" class="0">
 <segment>
-<pinref part="U$1" gate="G$1" pin="MISO"/>
-<wire x1="-53.34" y1="-124.46" x2="-68.58" y2="-124.46" width="0.1524" layer="91"/>
-<label x="-68.58" y="-124.46" size="1.778" layer="95"/>
+<wire x1="-53.34" y1="-114.3" x2="-73.66" y2="-114.3" width="0.1524" layer="91"/>
+<label x="-73.66" y="-114.3" size="1.778" layer="95"/>
+<pinref part="U11" gate="G$1" pin="SDO"/>
 </segment>
 <segment>
@@
 </segment>
 <segment>
-<pinref part="U$1" gate="G$1" pin="MOSI"/>
-<wire x1="-53.34" y1="-129.54" x2="-68.58" y2="-129.54" width="0.1524" layer="91"/>
-<label x="-68.58" y="-129.54" size="1.778" layer="95"/>
+<wire x1="-53.34" y1="-116.84" x2="-73.66" y2="-116.84" width="0.1524" layer="91"/>
+<label x="-73.66" y="-116.84" size="1.778" layer="95"/>
+<pinref part="U11" gate="G$1" pin="SDI"/>
 </segment>
 </net>
@@
 </segment>
 <segment>
-<pinref part="U$1" gate="G$1" pin="SCK"/>
-<wire x1="-53.34" y1="-119.38" x2="-68.58" y2="-119.38" width="0.1524" layer="91"/>
-<label x="-68.58" y="-119.38" size="1.778" layer="95"/>
+<wire x1="-53.34" y1="-111.76" x2="-73.66" y2="-111.76" width="0.1524" layer="91"/>
+<label x="-73.66" y="-111.76" size="1.778" layer="95"/>
+<pinref part="U11" gate="G$1" pin="SCK"/>
 </segment>
 </net>
@@
 </segment>
 <segment>
-<pinref part="U$1" gate="G$1" pin="CS"/>
-<wire x1="-53.34" y1="-114.3" x2="-68.58" y2="-114.3" width="0.1524" layer="91"/>
-<label x="-68.58" y="-114.3" size="1.778" layer="95"/>
+<label x="-73.66" y="-109.22" size="1.778" layer="95"/>
+<wire x1="-53.34" y1="-109.22" x2="-73.66" y2="-109.22" width="0.1524" layer="91"/>
+<pinref part="U11" gate="G$1" pin="CS"/>
 </segment>
 </net>
@@
 </segment>
 <segment>
-<pinref part="U$1" gate="G$1" pin="SCL"/>
-<wire x1="-15.24" y1="-124.46" x2="0" y2="-124.46" width="0.1524" layer="91"/>
-<label x="0" y="-124.46" size="1.778" layer="95"/>
+<wire x1="-20.32" y1="-111.76" x2="0" y2="-111.76" width="0.1524" layer="91"/>
+<label x="0" y="-111.76" size="1.778" layer="95"/>
+<pinref part="U11" gate="G$1" pin="SCL"/>
 </segment>
 </net>
@@
 </segment>
 <segment>
-<pinref part="U$1" gate="G$1" pin="SDA"/>
-<wire x1="-15.24" y1="-129.54" x2="0" y2="-129.54" width="0.1524" layer="91"/>
-<label x="0" y="-129.54" size="1.778" layer="95"/>
+<wire x1="-20.32" y1="-109.22" x2="0" y2="-109.22" width="0.1524" layer="91"/>
+<label x="0" y="-109.22" size="1.778" layer="95"/>
+<pinref part="U11" gate="G$1" pin="SDA"/>
 </segment>
 </net>
@@
 </segment>
 <segment>
-<pinref part="U$1" gate="G$1" pin="INT"/>
-<wire x1="-15.24" y1="-109.22" x2="0" y2="-109.22" width="0.1524" layer="91"/>
-<label x="0" y="-109.22" size="1.778" layer="95"/>
+<wire x1="-20.32" y1="-119.38" x2="0" y2="-119.38" width="0.1524" layer="91"/>
+<label x="0" y="-119.38" size="1.778" layer="95"/>
+<pinref part="U11" gate="G$1" pin="INT"/>
 </segment>
 </net>
@@
 </segment>
 <segment>
-<pinref part="U$1" gate="G$1" pin="PWM"/>
-<wire x1="-15.24" y1="-104.14" x2="0" y2="-104.14" width="0.1524" layer="91"/>
-<label x="0" y="-104.14" size="1.778" layer="95"/>
+<wire x1="-17.78" y1="-121.92" x2="0" y2="-121.92" width="0.1524" layer="91"/>
+<label x="0" y="-121.92" size="1.778" layer="95"/>
 </segment>
 </net>
@@
 <net name="LPUART0_RX_MKB" class="0">
 <segment>
-<pinref part="U$1" gate="G$1" pin="RX"/>
-<wire x1="-15.24" y1="-114.3" x2="0" y2="-114.3" width="0.1524" layer="91"/>
+<wire x1="-20.32" y1="-114.3" x2="0" y2="-114.3" width="0.1524" layer="91"/>
 <label x="0" y="-114.3" size="1.778" layer="95"/>
+<pinref part="U11" gate="G$1" pin="RX"/>
 </segment>
 <segment>
@@
 <net name="LPUART0_TX_MKB" class="0">
 <segment>
-<pinref part="U$1" gate="G$1" pin="TX"/>
-<wire x1="-15.24" y1="-119.38" x2="0" y2="-119.38" width="0.1524" layer="91"/>
-<label x="0" y="-119.38" size="1.778" layer="95"/>
-</segment>
-<segment>
+<wire x1="-20.32" y1="-116.84" x2="0" y2="-116.84" width="0.1524" layer="91"/>
+<label x="0" y="-116.84" size="1.778" layer="95"/>
+<pinref part="U11" gate="G$1" pin="TX"/>
+</segment>
+<segment>

Commit message: Práctica 1 - Entregada y Corregida
Con todos sus valores adecuados, esquematico y PCB, solo faltó ROUTEAR adecuadamente con criterios como estabilidad en las fuentes y demas.
Parts:
- added LED4, LED5: (no value), led:LED5MM
- R11, R9: value 130 -> 1k
- R5, R7: value 10K -> 1K
Connections:
- new net N$59: LED4.A, R7.2
- new net N$60: LED5.A, R5.2
- net +5V: now also U13.VDD
- net GND: now also LED4.C, LED5.C, U13.GND; no longer R5.2, R7.2
Changed lines of the file:
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@@
 <part name="+3V3" library="supply2" library_urn="urn:adsk.eagle:library:372" deviceset="+5V" device="" value="+3V3"/>
 <part name="R4" library="rcl" library_urn="urn:adsk.eagle:library:334" deviceset="R-US_" device="0309/12" package3d_urn="urn:adsk.eagle:package:23571/1" value="10K"/>
-<part name="R5" library="rcl" library_urn="urn:adsk.eagle:library:334" deviceset="R-US_" device="0309/12" package3d_urn="urn:adsk.eagle:package:23571/1" value="10K"/>
+<part name="R5" library="rcl" library_urn="urn:adsk.eagle:library:334" deviceset="R-US_" device="0309/12" package3d_urn="urn:adsk.eagle:package:23571/1" value="1K"/>
 <part name="CARGA" library="con-ptr500" library_urn="urn:adsk.eagle:library:181" deviceset="AK300/2" device="" package3d_urn="urn:adsk.eagle:package:9881/1"/>
 <part name="+24V" library="con-ptr500" library_urn="urn:adsk.eagle:library:181" deviceset="AK300/2" device="" package3d_urn="urn:adsk.eagle:package:9881/1"/>
@@
 <part name="Q2" library="IRF7416PBF_Completo" deviceset="IRF7416PBF" device=""/>
 <part name="R6" library="rcl" library_urn="urn:adsk.eagle:library:334" deviceset="R-US_" device="0309/12" package3d_urn="urn:adsk.eagle:package:23571/1" value="10K"/>
-<part name="R7" library="rcl" library_urn="urn:adsk.eagle:library:334" deviceset="R-US_" device="0309/12" package3d_urn="urn:adsk.eagle:package:23571/1" value="10K"/>
+<part name="R7" library="rcl" library_urn="urn:adsk.eagle:library:334" deviceset="R-US_" device="0309/12" package3d_urn="urn:adsk.eagle:package:23571/1" value="1K"/>
 <part name="CARGA2" library="con-ptr500" library_urn="urn:adsk.eagle:library:181" deviceset="AK300/2" device="" package3d_urn="urn:adsk.eagle:package:9881/1"/>
 <part name="+24V1" library="con-ptr500" library_urn="urn:adsk.eagle:library:181" deviceset="AK300/2" device="" package3d_urn="urn:adsk.eagle:package:9881/1"/>
@@
 <part name="INPUT1" library="con-ptr500" library_urn="urn:adsk.eagle:library:181" deviceset="AK300/2" device="" package3d_urn="urn:adsk.eagle:package:9881/1"/>
 <part name="R10" library="rcl" library_urn="urn:adsk.eagle:library:334" deviceset="R-US_" device="0204/7" package3d_urn="urn:adsk.eagle:package:23498/1" value="220"/>
-<part name="R11" library="rcl" library_urn="urn:adsk.eagle:library:334" deviceset="R-US_" device="0309/12" package3d_urn="urn:adsk.eagle:package:23571/1" value="130"/>
+<part name="R11" library="rcl" library_urn="urn:adsk.eagle:library:334" deviceset="R-US_" device="0309/12" package3d_urn="urn:adsk.eagle:package:23571/1" value="1k"/>
 <part name="LED1" library="led" library_urn="urn:adsk.eagle:library:259" deviceset="LED" device="5MM" package3d_urn="urn:adsk.eagle:package:15799/2"/>
 <part name="R12" library="rcl" library_urn="urn:adsk.eagle:library:334" deviceset="R-US_" device="0204/7" package3d_urn="urn:adsk.eagle:package:23498/1" value="10K"/>
@@
 <part name="INPUT2" library="con-ptr500" library_urn="urn:adsk.eagle:library:181" deviceset="AK300/2" device="" package3d_urn="urn:adsk.eagle:package:9881/1"/>
 <part name="R8" library="rcl" library_urn="urn:adsk.eagle:library:334" deviceset="R-US_" device="0309/12" package3d_urn="urn:adsk.eagle:package:23571/1" value="220"/>
-<part name="R9" library="rcl" library_urn="urn:adsk.eagle:library:334" deviceset="R-US_" device="0309/12" package3d_urn="urn:adsk.eagle:package:23571/1" value="130"/>
+<part name="R9" library="rcl" library_urn="urn:adsk.eagle:library:334" deviceset="R-US_" device="0309/12" package3d_urn="urn:adsk.eagle:package:23571/1" value="1k"/>
 <part name="LED2" library="led" library_urn="urn:adsk.eagle:library:259" deviceset="LED" device="5MM" package3d_urn="urn:adsk.eagle:package:15799/2"/>
 <part name="R13" library="rcl" library_urn="urn:adsk.eagle:library:334" deviceset="R-US_" device="0204/7" package3d_urn="urn:adsk.eagle:package:23498/1" value="10K"/>
@@
 <part name="GND49" library="supply1" library_urn="urn:adsk.eagle:library:371" deviceset="GND" device=""/>
 <part name="U11" library="MIKROE-971" deviceset="MIKROE-971" device=""/>
+<part name="GND13" library="supply1" library_urn="urn:adsk.eagle:library:371" deviceset="GND" device=""/>
+<part name="LED4" library="led" library_urn="urn:adsk.eagle:library:259" deviceset="LED" device="5MM" package3d_urn="urn:adsk.eagle:package:15799/2"/>
+<part name="LED5" library="led" library_urn="urn:adsk.eagle:library:259" deviceset="LED" device="5MM" package3d_urn="urn:adsk.eagle:package:15799/2"/>
 </parts>
 <sheets>
@@
 <instance part="+5V" gate="1" x="-48.26" y="177.8" rot="R270"/>
 <instance part="GND46" gate="1" x="-76.2" y="154.94"/>
-<instance part="GND47" gate="1" x="-2.54" y="27.94"/>
-<instance part="GND48" gate="1" x="-190.5" y="30.48"/>
+<instance part="GND47" gate="1" x="2.54" y="15.24"/>
+<instance part="GND48" gate="1" x="-182.88" y="17.78"/>
 <instance part="GND8" gate="1" x="-68.58" y="-76.2"/>
 <instance part="GND9" gate="1" x="104.14" y="-73.66"/>
@@
 <instance part="GND49" gate="1" x="429.26" y="-327.66"/>
 <instance part="U11" gate="G$1" x="-53.34" y="-104.14"/>
+<instance part="GND13" gate="1" x="535.94" y="127"/>
+<instance part="LED4" gate="G$1" x="-182.88" y="33.02"/>
+<instance part="LED5" gate="G$1" x="2.54" y="30.48"/>
 </instances>
 <busses>
@@
 </segment>
 <segment>
-<pinref part="GND48" gate="1" pin="GND"/>
-<pinref part="R7" gate="G$1" pin="2"/>
-<wire x1="-190.5" y1="33.02" x2="-190.5" y2="40.64" width="0.1524" layer="91"/>
-<wire x1="-190.5" y1="40.64" x2="-180.34" y2="40.64" width="0.1524" layer="91"/>
-</segment>
-<segment>
-<pinref part="GND47" gate="1" pin="GND"/>
-<pinref part="R5" gate="G$1" pin="2"/>
-<wire x1="-2.54" y1="30.48" x2="-2.54" y2="38.1" width="0.1524" layer="91"/>
-<wire x1="-2.54" y1="38.1" x2="5.08" y2="38.1" width="0.1524" layer="91"/>
-</segment>
-<segment>
 <pinref part="U6" gate="A" pin="E"/>
 <wire x1="-78.74" y1="-66.04" x2="-68.58" y2="-66.04" width="0.1524" layer="91"/>
@@
 <wire x1="429.26" y1="-322.58" x2="429.26" y2="-325.12" width="0.1524" layer="91"/>
 <pinref part="GND49" gate="1" pin="GND"/>
+</segment>
+<segment>
+<pinref part="U13" gate="A" pin="GND"/>
+<wire x1="528.32" y1="129.54" x2="535.94" y2="129.54" width="0.1524" layer="91"/>
+<pinref part="GND13" gate="1" pin="GND"/>
+</segment>
+<segment>
+<pinref part="LED4" gate="G$1" pin="C"/>
+<pinref part="GND48" gate="1" pin="GND"/>
+<wire x1="-182.88" y1="27.94" x2="-182.88" y2="20.32" width="0.1524" layer="91"/>
+</segment>
+<segment>
+<pinref part="LED5" gate="G$1" pin="C"/>
+<pinref part="GND47" gate="1" pin="GND"/>
+<wire x1="2.54" y1="25.4" x2="2.54" y2="17.78" width="0.1524" layer="91"/>
 </segment>
 </net>
@@
 <label x="0" y="-106.68" size="1.778" layer="95"/>
 <pinref part="U11" gate="G$1" pin="5V"/>
+</segment>
+<segment>
+<pinref part="U13" gate="A" pin="VDD"/>
+<wire x1="472.44" y1="129.54" x2="467.36" y2="129.54" width="0.1524" layer="91"/>
+<label x="464.82" y="129.54" size="1.778" layer="95"/>
 </segment>
 </net>
@@
 </segment>
 </net>
+<net name="N$59" class="0">
+<segment>
+<pinref part="R7" gate="G$1" pin="2"/>
+<wire x1="-180.34" y1="40.64" x2="-182.88" y2="40.64" width="0.1524" layer="91"/>
+<pinref part="LED4" gate="G$1" pin="A"/>
+<wire x1="-182.88" y1="40.64" x2="-182.88" y2="35.56" width="0.1524" layer="91"/>
+</segment>
+</net>
+<net name="N$60" class="0">
+<segment>
+<pinref part="R5" gate="G$1" pin="2"/>
+<wire x1="5.08" y1="38.1" x2="2.54" y2="38.1" width="0.1524" layer="91"/>
+<pinref part="LED5" gate="G$1" pin="A"/>
+<wire x1="2.54" y1="38.1" x2="2.54" y2="33.02" width="0.1524" layer="91"/>
+</segment>
+</net>
